File: chain-item.sch (KiCad schematic (older format))
At the start: 17 parts, among them CON1 AVR-ISP-6, J1 Conn_01x04, J2 R_PAD1, J3 R_PAD2, J4 Conn_01x04, J5 R_PAD1, J6 R_PAD2, U1 ATTINY10-TS

Commit message: Add description and version
Parts:
- J2, J3: footprint chain-item:pad_resistor -> chain-item:pogopin
- J5, J6: footprint Measurement_Points:Measurement_Point_Round-SMD-Pad_Big -> chain-item:pad_resistor
Changed lines of the file:
@@
 encoding utf-8
 Sheet 1 1
-Title ""
-Date ""
-Rev ""
+Title "ACC - Chain Item "
+Date "2018-05-01"
+Rev "v1"
 Comp ""
 Comment1 ""
@@
 F 0 "J2" H 3150 6250 50  0000 C CNN
 F 1 "R_PAD1" H 3350 6200 50  0000 C CNN
-F 2 "chain-item:pad_resistor" H 3200 6200 50  0001 C CNN
+F 2 "chain-item:pogopin" H 3200 6200 50  0001 C CNN
 F 3 "~" H 3200 6200 50  0001 C CNN
 	1    3200 6200
@@
 F 0 "J3" H 3150 6500 50  0000 C CNN
 F 1 "R_PAD2" H 3350 6450 50  0000 C CNN
-F 2 "chain-item:pad_resistor" H 3200 6450 50  0001 C CNN
+F 2 "chain-item:pogopin" H 3200 6450 50  0001 C CNN
 F 3 "~" H 3200 6450 50  0001 C CNN
 	1    3200 6450
@@
 F 0 "J5" H 2072 6030 50  0000 R CNN
 F 1 "R_PAD1" H 2072 6121 50  0000 R CNN
-F 2 "Measurement_Points:Measurement_Point_Round-SMD-Pad_Big" H 2100 6100 50  0001 C CNN
+F 2 "chain-item:pad_resistor" H 2100 6100 50  0001 C CNN
 F 3 "~" H 2100 6100 50  0001 C CNN
 	1    2100 6100
@@
 F 0 "J6" H 2072 6530 50  0000 R CNN
 F 1 "R_PAD2" H 2072 6621 50  0000 R CNN
-F 2 "Measurement_Points:Measurement_Point_Round-SMD-Pad_Big" H 2100 6600 50  0001 C CNN
+F 2 "chain-item:pad_resistor" H 2100 6600 50  0001 C CNN
 F 3 "~" H 2100 6600 50  0001 C CNN
 	1    2100 6600
